File: motorstyrning.brd (EAGLE design)
At the start: 25 parts

Commit message: added .pyc and .b#1 files to gitignore, updated pcb layout to latest version
Routing:
- net S$22: track 4.34 -> 3.17 mm
- net S$13: track 7.78 -> 6.81 mm
- net S$20: track 36.4 -> 35.7 mm
- net S$14: track 5.61 -> 4.94 mm
- net S$21: track 6.66 -> 6.03 mm
- net S$23: track 53.2 -> 52.7 mm
- net S$3: track 58.4 -> 57.9 mm
- added copper zone on layer 16, net S$27
Other:
- board text added: "A"
- board text added: "B"
- board text added: "C"
- board text added: "Engine"
- board text added: "LED1"
- board text added: "LED2"
- board text added: "LED3"
- board text added: "LED4"
- board text added: "Robotstyrning Layout Daniel Häggmyr"
- board text added: "Steering"
- board text removed: "(~'-')~"
Changed lines of the file:
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@@
 <setting verticaltext="up"/>
 </settings>
-<grid distance="0.05" unitdist="inch" unit="inch" style="lines" multiple="1" display="no" altdistance="0.025" altunitdist="inch" altunit="inch"/>
+<grid distance="0.005" unitdist="inch" unit="inch" style="lines" multiple="1" display="no" altdistance="0.025" altunitdist="inch" altunit="inch"/>
 <layers>
 <layer number="1" name="Top" color="4" fill="1" visible="yes" active="yes"/>
@@
 <layer number="19" name="Unrouted" color="6" fill="1" visible="yes" active="yes"/>
 <layer number="20" name="Dimension" color="15" fill="1" visible="no" active="yes"/>
-<layer number="21" name="tPlace" color="7" fill="1" visible="yes" active="yes"/>
-<layer number="22" name="bPlace" color="7" fill="1" visible="yes" active="yes"/>
-<layer number="23" name="tOrigins" color="15" fill="1" visible="yes" active="yes"/>
-<layer number="24" name="bOrigins" color="15" fill="1" visible="yes" active="yes"/>
+<layer number="21" name="tPlace" color="7" fill="1" visible="no" active="yes"/>
+<layer number="22" name="bPlace" color="7" fill="1" visible="no" active="yes"/>
+<layer number="23" name="tOrigins" color="15" fill="1" visible="no" active="yes"/>
+<layer number="24" name="bOrigins" color="15" fill="1" visible="no" active="yes"/>
 <layer number="25" name="tNames" color="7" fill="1" visible="no" active="yes"/>
 <layer number="26" name="bNames" color="7" fill="1" visible="no" active="yes"/>
@@
 <hole x="55" y="40" drill="3.2"/>
 <hole x="5" y="40" drill="3.2"/>
-<text x="4.445" y="10.16" size="1.778" layer="16">(~'-')~</text>
-<text x="9.525" y="14.605" size="1.778" layer="16" rot="MR0">(~'-')~</text>
+<text x="12.7" y="12.7" size="1.016" layer="16" font="vector" rot="MR180">Robotstyrning
+Layout Daniel Häggmyr</text>
+<text x="56.515" y="26.924" size="1.016" layer="16" font="vector" rot="MR90">Engine</text>
+<text x="49.149" y="42.291" size="1.016" layer="16" font="vector" rot="MR0">Steering</text>
+<text x="49.403" y="39.497" size="1.016" layer="16" font="vector" rot="MR270">LED1</text>
+<text x="47.879" y="21.971" size="1.016" layer="16" font="vector" rot="MR90">LED2</text>
+<text x="19.939" y="2.032" size="1.016" layer="16" font="vector" rot="MR0">LED3</text>
+<text x="3.937" y="2.032" size="1.016" layer="16" font="vector" rot="MR0">LED4</text>
+<text x="30.988" y="37.465" size="1.016" layer="16" font="vector" rot="MR0">A</text>
+<text x="40.005" y="32.512" size="1.016" layer="16" font="vector" rot="MR0">A</text>
+<text x="23.368" y="37.338" size="1.016" layer="16" font="vector" rot="MR0">B</text>
+<text x="57.531" y="19.812" size="1.016" layer="16" font="vector" rot="MR0">B</text>
+<text x="15.875" y="37.338" size="1.016" layer="16" font="vector" rot="MR0">C</text>
+<text x="51.054" y="19.939" size="1.016" layer="16" font="vector" rot="MR0">C</text>
 </plain>
 <attributes>
@@
 </signal>
 <signal name="S$23">
-<wire x1="31.75" y1="20.32" x2="35.56" y2="24.13" width="0.4064" layer="16"/>
+<wire x1="32.131" y1="20.701" x2="35.56" y2="24.13" width="0.4064" layer="16"/>
 <contactref element="PNP1" pad="E"/>
 <wire x1="35.56" y1="24.13" x2="35.56" y2="29.21" width="0.4064" layer="16"/>
@@
 <signal name="S$13">
 <contactref element="E$10" pad="1"/>
-<wire x1="26.67" y1="20.32" x2="26.67" y2="22.86" width="0.4064" layer="16"/>
-<wire x1="26.67" y1="22.86" x2="31.75" y2="24.13" width="0.4064" layer="16"/>
+<wire x1="27.051" y1="20.828" x2="27.051" y2="22.733" width="0.4064" layer="16"/>
+<wire x1="27.051" y1="22.733" x2="31.75" y2="24.13" width="0.4064" layer="16"/>
 </signal>
 <signal name="S$14">
-<wire x1="21.59" y1="20.32" x2="21.59" y2="22.86" width="0.4064" layer="16"/>
-<wire x1="21.59" y1="22.86" x2="22.86" y2="24.13" width="0.4064" layer="16"/>
+<wire x1="21.971" y1="20.828" x2="21.971" y2="23.241" width="0.4064" layer="16"/>
+<wire x1="21.971" y1="23.241" x2="22.86" y2="24.13" width="0.4064" layer="16"/>
 <contactref element="E$11" pad="1"/>
 <wire x1="22.86" y1="24.13" x2="24.13" y2="24.13" width="0.4064" layer="16"/>
 </signal>
 <signal name="S$15">
-<wire x1="19.05" y1="21.59" x2="16.51" y2="24.13" width="0.4064" layer="16"/>
+<wire x1="19.304" y1="21.336" x2="16.51" y2="24.13" width="0.4064" layer="16"/>
 <contactref element="E$12" pad="1"/>
 </signal>
 <signal name="S$16">
-<wire x1="11.43" y1="21.59" x2="8.89" y2="24.13" width="0.4064" layer="16"/>
+<wire x1="11.684" y1="21.336" x2="8.89" y2="24.13" width="0.4064" layer="16"/>
 <contactref element="E$13" pad="1"/>
 </signal>
@@
 </signal>
 <signal name="S$20">
-<wire x1="36.83" y1="6.35" x2="31.75" y2="1.27" width="0.4064" layer="16"/>
-<wire x1="31.75" y1="1.27" x2="12.7" y2="1.27" width="0.4064" layer="16"/>
-<wire x1="12.7" y1="1.27" x2="5.08" y2="1.27" width="0.4064" layer="16"/>
-<wire x1="5.08" y1="1.27" x2="5.08" y2="2.54" width="0.4064" layer="16"/>
-<wire x1="12.7" y1="2.54" x2="12.7" y2="1.27" width="0.4064" layer="16"/>
+<wire x1="36.957" y1="5.334" x2="32.893" y2="1.27" width="0.4064" layer="16"/>
+<wire x1="32.893" y1="1.27" x2="12.954" y2="1.27" width="0.4064" layer="16"/>
+<wire x1="12.954" y1="1.27" x2="5.334" y2="1.27" width="0.4064" layer="16"/>
+<wire x1="5.334" y1="1.27" x2="5.334" y2="2.413" width="0.4064" layer="16"/>
+<wire x1="12.954" y1="2.54" x2="12.954" y2="1.27" width="0.4064" layer="16"/>
 </signal>
 <signal name="S$21">
-<wire x1="12.7" y1="6.35" x2="8.89" y2="2.54" width="0.4064" layer="16"/>
+<wire x1="12.319" y1="5.842" x2="8.89" y2="2.54" width="0.4064" layer="16"/>
 <wire x1="8.89" y1="2.54" x2="7.62" y2="2.54" width="0.4064" layer="16"/>
 </signal>
 <signal name="S$22">
-<wire x1="13.97" y1="6.35" x2="15.24" y2="5.08" width="0.4064" layer="16"/>
-<wire x1="15.24" y1="5.08" x2="15.24" y2="2.54" width="0.4064" layer="16"/>
+<wire x1="14.351" y1="5.588" x2="14.986" y2="4.064" width="0.4064" layer="16"/>
+<wire x1="14.986" y1="4.064" x2="14.986" y2="2.54" width="0.4064" layer="16"/>
 </signal>
 <signal name="S$18">
@@
 <wire x1="15.875" y1="43.815" x2="23.495" y2="43.815" width="0.4064" layer="16"/>
 <wire x1="23.495" y1="43.815" x2="31.115" y2="43.815" width="0.4064" layer="16"/>
-<wire x1="31.115" y1="43.815" x2="41.275" y2="43.815" width="0.4064" layer="16"/>
+<wire x1="31.115" y1="43.815" x2="41.021" y2="43.815" width="0.4064" layer="16"/>
 <wire x1="20.32" y1="39.37" x2="23.495" y2="39.37" width="0.4064" layer="16"/>
 <wire x1="23.495" y1="39.37" x2="23.495" y2="43.815" width="0.4064" layer="16"/>
-<wire x1="35.56" y1="39.37" x2="41.275" y2="39.37" width="0.4064" layer="16"/>
-<wire x1="41.275" y1="39.37" x2="41.275" y2="43.815" width="0.4064" layer="16"/>
+<wire x1="35.56" y1="39.37" x2="41.021" y2="39.37" width="0.4064" layer="16"/>
+<wire x1="41.021" y1="39.37" x2="41.021" y2="43.815" width="0.4064" layer="16"/>
 <wire x1="27.94" y1="39.37" x2="31.115" y2="39.37" width="0.4064" layer="16"/>
 <wire x1="31.115" y1="39.37" x2="31.115" y2="43.815" width="0.4064" layer="16"/>
+</signal>
+<signal name="S$27">
+<polygon width="0.4064" layer="16" spacing="0.254" pour="cutout" isolate="0.3048">
+<vertex x="11.303" y="9.271"/>
+<vertex x="11.303" y="13.843"/>
+<vertex x="32.893" y="13.843"/>
+<vertex x="32.893" y="8.89"/>
+<vertex x="11.303" y="8.89"/>
+</polygon>
 </signal>
 </signals>
 </board>
 </drawing>
+<compatibility>
+<note version="6.3" minversion="6.2.2" severity="warning">
+Since Version 6.2.2 text objects can contain more than one line,
+which will not be processed correctly with this version.
+</note>
+</compatibility>
 </eagle>
